File: hardware/circuit-boards/dual-converter-boost-converter-module-V1.0/dual-converter-boost-converter-module-V1.0.kicad_sch (KiCad schematic)
At the start: 46 parts, among them J1 Vout Conn, J2 Conn_01x06, J3 Vout Conn, U1 TPL0401B-10DCKR, U2 LM5156HPWPR, U3 STN3N40K3

Commit message: update decals
Other:
- company: Rack Robotics, Inc. -> EPL Capstone 2026
