File: hardware/circuit-boards/dual-converter-motherboard-V1.0/dual-converter-motherboard-V1.0.kicad_pcb (KiCad board)
At the start: 6 copper layers, 230 x 76 mm, 107 parts, among them J1 2601-1102, J10 Conn_02x03_Odd_Even, J11 Conn_01x06_Socket, J12 Conn_02x03_Odd_Even, J13 Conn_02x03_Odd_Even, J14 Conn_02x03_Odd_Even, J15 Conn_01x06_Socket, J16 Conn_01x07_Socket, J2 2601-1102, J3 S4B-XH-SM4-TB, J4 Conn_02x03_Odd_Even, J5 Conn_02x03_Odd_Even, J6 Conn_02x03_Odd_Even, J7 Conn_02x03_Odd_Even, J8 Conn_02x03_Odd_Even, J9 Conn_02x03_Odd_Even, Q1 SUM110P08-11L-E3, Q2 DMP45H4D9HK3-13, Q3 SIHB068N60EF-GE3, U4 UCC23313BDWYR, U5 TMCS1133C1A, U6 UCC23313BDWYR, U7 UCC23313BDWYR, U8 SC0915

Commit message: update decals
Other:
- board text added: "Based on Powercore V3 by RackRobotics"
- board text added: "SPARKEDM"
- board text removed: "DESIGNED BY"
- board text removed: "POWERCORE V3-EPL"
- board text removed: "RACK ROBOTICS"
