File: hardware/circuit-boards/dual-converter-motherboard-V1.0/dual-converter-motherboard-V1.0.kicad_sch (KiCad schematic)
At the start: 45 parts, among them J1 2601-1102, J10 Conn_02x03_Odd_Even, J11 Conn_01x06_Socket, J12 Conn_02x03_Odd_Even, J13 Conn_02x03_Odd_Even, J14 Conn_02x03_Odd_Even, J15 Conn_01x06_Socket, J16 Conn_01x07_Socket, J2 2601-1102, J3 S4B-XH-SM4-TB, J4 Conn_02x03_Odd_Even, J5 Conn_02x03_Odd_Even, J6 Conn_02x03_Odd_Even, J7 Conn_02x03_Odd_Even, J8 Conn_02x03_Odd_Even, J9 Conn_02x03_Odd_Even, U1 POWER_MANAGEMENT_MODULE, U2 HIGH-CURRENT_PHASE_MODULE_V1.0, U3 HIGH-VOLTAGE_PHASE_MODULE

Commit message: update decals
Other:
- company: Rack Robotics, Inc. -> EPL Capstone 2026
