File: hardware/circuit-boards/dual-converter-pi-filter-module-V1.0/buck-converter.kicad_sch (KiCad schematic)
At the start: 64 parts, among them Q1 BSZ070N08LS5ATMA1, Q2 BSZ070N08LS5ATMA1, U1 TPL0401B-10DCKR, U2 LM5149-Q1

Commit message: update decals
Other:
- company: Rack Robotics, Inc. -> EPL Capstone 2026
