File: hardware/circuit-boards/dual-converter-pi-filter-module-V1.0/dual-converter-pi-filter-module-V1.0.kicad_sch (KiCad schematic)
At the start: 52 parts

Commit message: update decals
Other:
- company: Rack Robotics, Inc. -> EPL Capstone 2026
