File: hardware/circuit-boards/dual-converter-power-management-module-V1.0/dual-converter-power-management-module-V1.0.kicad_sch (KiCad schematic)
At the start: 60 parts, among them J1 Conn_02x03_Odd_Even, J2 Conn_01x06_Pin, J3 Conn_02x03_Odd_Even, J4 Conn_02x03_Odd_Even, J5 Conn_02x03_Odd_Even, U1 TPS1HTC30AQPWPRQ1

Commit message: update decals
Other:
- company: Rack Robotics, Inc. -> EPL Capstone 2026
